Commit message: init

File: basic_mobile_robot3/models/basic_mobile_bot_v2.urdf (robot description, URDF)
Before this commit: robot basic_mobile_bot, 6 links, 9 joints
Links:
- added link rgb_cam_camera_link; visual box size=0.02 0.04 0.01
- added link rgb_cam_camera_link_frame
- link base_link: geometry collision box size=${base_length} ${base_width} ${base_height}; visual mesh filename=package://basic_mobile_robot3/meshes/base_link.dae
- link fork: geometry collision mesh filename=package://basic_mobile_robot3/meshes/fork.dae; visual mesh filename=package://basic_mobile_robot3/meshes/fork.dae
Joints:
- added joint rgb_cam_camera_frame_joint: type fixed, parent rgb_cam_camera_link, child rgb_cam_camera_link_frame, origin xyz=0.01 0 0 rpy=0 0 0, axis 0 0 0
- added joint rgb_cam_camera_link_joint: type fixed, parent base_link, child rgb_cam_camera_link, origin xyz=0.04 0.0 0.5 rpy=0 0 0
